Commit message: add 502 model

File: iqr_4b_robot-master/iqr_4b_description/urdf/iqr_4b_robot.urdf.xacro (robot description, xacro)
@@ -25,5 +25,5 @@
   <!-- IQR pan-tilt -->
   <xacro:pan_tilt parent="jackal_support_link">
-    <origin xyz="-0.0801 0 0.628" rpy="0 0 0" />
+    <origin xyz="-0.0801 0 1.128" rpy="0 0 0" />
   </xacro:pan_tilt>
   <!-- Kinect v2 -->
@@ -36,6 +36,6 @@
 	    <updateRate>50.0</updateRate>
 	    <bodyName>base_link</bodyName>
-	    <topicName>ground_truth/state</topicName>
-	    <gaussianNoise>0.01</gaussianNoise>
+	    <topicName>ground_truth/robot_state</topicName>
+	    <gaussianNoise>0.00</gaussianNoise>
 	    <frameName>world</frameName>
 	    <xyzOffsets>0 0 0</xyzOffsets>

File: iqr_4b_robot-master/iqr_4b_description/urdf/kinect_v2.xacro (robot description, xacro)
@@ -39,5 +39,5 @@
           <clip>
             <near>0.05</near>
-            <far>8.0</far>
+            <far>16</far>
           </clip>
         </camera>

File: iqr_4b_robot-master/iqr_4b_description/urdf/vlp16.xacro (robot description, xacro)
@@ -3,26 +3,9 @@
   <xacro:macro name="vlp16" params="package parent *origin">
     <xacro:property name="prefix" value="vlp16"/>
-    <link name="${prefix}_link">
-      <visual>
-        <origin xyz="0 0 0" rpy="0 0 0"/>
-        <geometry>
-          <mesh filename="package://${package}/urdf/mesh/VLP16.stl"/>
-        </geometry>
-        <material name="">
-          <color rgba="1.0 1.0 0.9 1"/>
-        </material>
-      </visual>
-    </link>
-    <joint name="${prefix}_link_joint" type="fixed">
-      <xacro:insert_block name="origin"/>
-      <parent link="${parent}"/>
-      <child link="${prefix}_link"/>
-    </joint>
-    <link name="velodyne"/>
-    <joint name="velodyne_link_joint" type="fixed">
-      <origin xyz="0 0 0.040" rpy="0 0 0" />
-      <parent link="${prefix}_link"/>
-      <child link="velodyne"/>
-    </joint>
+	 <!-- VLP-16 -->
+	  <xacro:include filename="$(find velodyne_description)/urdf/VLP-16.urdf.xacro"/>
+	  <VLP-16 parent="${parent}" name="velodyne" topic="/velodyne_points" hz="10" samples="1024" gpu="false" lasers="16" max_range="100">
+	    <origin xyz="0 0 0" rpy="0 0 0" />
+	  </VLP-16>
   </xacro:macro>
 </robot>

File: iqr_4b_robot-master/iqr_4b_description/urdf/zed.xacro (robot description, xacro)
@@ -19,4 +19,51 @@
       <child link="${prefix}_link"/>
     </joint>
+	  <!-- stereo camera >
+    <gazebo reference="${prefix}_link">
+      <sensor type="multicamera" name="stereocamera">
+        <always_on>true</always_on>
+        <update_rate>10</update_rate>
+        <visualize>false</visualize>
+        <camera name="left">
+          <pose>0 0 0 0 0 0</pose>
+          <horizontal_fov>1.047</horizontal_fov>
+          <image>
+            <width>320</width>
+            <height>240</height>
+          </image>
+          <clip>
+            <near>0.1</near>
+            <far>100</far>
+          </clip>
+        </camera>
+        <camera name="right">
+          <pose>0 -0.07 0 0 0 0</pose>
+          <horizontal_fov>1.047</horizontal_fov>
+          <image>
+            <width>320</width>
+            <height>240</height>
+          </image>
+          <clip>
+            <near>0.1</near>
+            <far>100</far>
+          </clip>
+        </camera>
+        <plugin name="stereo_camera_controller" filename="libgazebo_ros_multicamera.so">
+          <cameraName>stereocamera</cameraName>
+          <alwaysOn>true</alwaysOn>
+          <updateRate>10</updateRate>
+          <cameraName>stereocamera</cameraName>
+          <imageTopicName>image_raw</imageTopicName>
+          <cameraInfoTopicName>camera_info</cameraInfoTopicName>
+          <frameName>camera_link_optical</frameName>
+          <baseline>0.07</baseline>
+          <distortion_k1>0.0</distortion_k1>
+          <distortion_k2>0.0</distortion_k2>
+          <distortion_k3>0.0</distortion_k3>
+          <distortion_t1>0.0</distortion_t1>
+          <distortion_t2>0.0</distortion_t2>
+        </plugin>
+      </sensor>
+    </gazebo-->
   </xacro:macro>
 </robot>

Commit message: change kinect orient

File: iqr_4b_robot-master/iqr_4b_description/urdf/iqr_4b_robot.urdf.xacro (robot description, xacro)
@@ -25,5 +25,5 @@
   <!-- IQR pan-tilt -->
   <xacro:pan_tilt parent="jackal_support_link">
-    <origin xyz="-0.0801 0 1.128" rpy="0 0 0" />
+    <origin xyz="-0.0801 0 0.625" rpy="0 0 0" />
   </xacro:pan_tilt>
   <!-- Kinect v2 -->

File: iqr_4b_robot-master/iqr_4b_description/urdf/vlp16.xacro (robot description, xacro)
@@ -6,5 +6,5 @@
 	  <xacro:include filename="$(find velodyne_description)/urdf/VLP-16.urdf.xacro"/>
 	  <VLP-16 parent="${parent}" name="velodyne" topic="/velodyne_points" hz="10" samples="1024" gpu="false" lasers="16" max_range="100">
-	    <origin xyz="0 0 0" rpy="0 0 0" />
+	    <xacro:insert_block name="origin" />
 	  </VLP-16>
   </xacro:macro>

Commit message: update

File: iqr_4b_robot-master/iqr_4b_description/urdf/iqr_4b_robot.urdf.xacro (robot description, xacro)
@@ -44,4 +44,4 @@
 	</gazebo>
   <!-- Kinova jaco j2n6s300 -->
-  <xacro:j2n6s300  base_parent="arm_mount_link"/>
+  <xacro:j2n6s300  base_parent="root"/>
 </robot>

File: iqr_4b_robot-master/iqr_4b_description/urdf/jackal_support.xacro (robot description, xacro)
@@ -19,9 +19,9 @@
       <child link="${prefix}_link"/>
     </joint>
-    <link name="arm_mount_link"/>
+    <link name="root"/>
     <joint name="arm_mount_link_joint" type="fixed">
       <origin xyz="-0.0460 0 0.07056" rpy="1.5707 0.0 1.5707" />
       <parent link="${prefix}_link"/>
-      <child link="arm_mount_link"/>
+      <child link="root"/>
     </joint>
   </xacro:macro>
