Commit message: solve wheel problem

File: asm_car_asm/urdf/asm_car_asm.urdf (robot description, URDF)
Before this commit: robot asm_car_asm, 18 links, 17 joints
Links:
- link base_link: mass 0.826691190957243 -> 30.826691190957243
- link body: mass 1.00302107294552 -> 10.00302107294552
- link rack_link: mass 6.56017677903339 -> 1.56017677903339

File: asm_car_asm/urdf/asm_car_asm.urdf.xacro (robot description, xacro)
@@ -31,6 +31,6 @@
 <gazebo reference="BackLeftWheel1">
 			<selfCollide>true</selfCollide>
-			<mu1 value="1.0"/>
-			<mu2 value="1.0"/>
+			<mu1 value="0.5"/>
+			<mu2 value="2"/>
 			<kp value="10000000.0" />
 			<kd value="1.0" />
@@ -40,6 +40,6 @@
 <gazebo reference="BackLeftWheel2">
 <selfCollide>true</selfCollide>
-			<mu1 value="1.0"/>
-			<mu2 value="1.0"/>
+			<mu1 value="0.5"/>
+			<mu2 value="2"/>
 			<kp value="10000000.0" />
 			<kd value="1.0" />
@@ -49,6 +49,6 @@
 <gazebo reference="FrontLeftWheel1">
 <selfCollide>true</selfCollide>
-			<mu1 value="1.0"/>
-			<mu2 value="1.0"/>
+			<mu1 value="0.5"/>
+			<mu2 value="2"/>
 			<kp value="10000000.0" />
 			<kd value="1.0" />
@@ -58,6 +58,6 @@
 <gazebo reference="FrontLeftWheel2">
 <selfCollide>true</selfCollide>
-			<mu1 value="1.0"/>
-			<mu2 value="1.0"/>
+			<mu1 value="0.5"/>
+			<mu2 value="2"/>
 			<kp value="10000000.0" />
 			<kd value="1.0" />
@@ -67,6 +67,6 @@
 <gazebo reference="BackRightWheel1">
 <selfCollide>true</selfCollide>
-			<mu1 value="1.0"/>
-			<mu2 value="1.0"/>
+			<mu1 value="0.5"/>
+			<mu2 value="2"/>
 			<kp value="10000000.0" />
 			<kd value="1.0" />
@@ -76,6 +76,6 @@
 <gazebo reference="BackRightWheel2">
 <selfCollide>true</selfCollide>
-			<mu1 value="1.0"/>
-			<mu2 value="1.0"/>
+			<mu1 value="0.5"/>
+			<mu2 value="2"/>
 			<kp value="10000000.0" />
 			<kd value="1.0" />
@@ -85,6 +85,6 @@
 <gazebo reference="FrontRightWheel1">
 <selfCollide>true</selfCollide>
-			<mu1 value="1.0"/>
-			<mu2 value="1.0"/>
+			<mu1 value="0.5"/>
+			<mu2 value="2"/>
 			<kp value="10000000.0" />
 			<kd value="1.0" />
@@ -94,6 +94,6 @@
 <gazebo reference="FrontRightWheel2">
 <selfCollide>true</selfCollide>
-			<mu1 value="1.0"/>
-			<mu2 value="1.0"/>
+			<mu1 value="0.5"/>
+			<mu2 value="2"/>
 			<kp value="10000000.0" />
 			<kd value="1.0" />

Commit message: add ur arm

File: asm_car_asm/urdf/asm_car_asm.urdf (robot description, URDF)
Before this commit: robot asm_car_asm, 18 links, 17 joints
Links:
- added link arm_base_link, mass 0.745925360702044; collision mesh filename=package://asm_car_asm/meshes/arm_base_link.STL; visual mesh filename=package://asm_car_asm/meshes/arm_base_link.STL
Joints:
- added joint ArmJoint: type fixed, parent body, child arm_base_link, origin xyz=-0.388 0 0 rpy=1.5708 0 0, axis 0 0 0
- added joint ur5_joint: type fixed, parent arm_base_link, child ur5_base_link, origin xyz=0.0 0.2 0.0 rpy=-1.5708 0.0 0.0
- joint kinect_joint: origin xyz=0 -0.12 0.653 rpy=0 0.7 -1.5708 -> xyz=0 0 0.603 rpy=0 0.7 -1.5708
- joint laser_joint: origin xyz=0 -0.12 0.693 rpy=0 0 -1.5708 -> xyz=0 0 0.653 rpy=0 0 -1.5708

File: asm_car_asm/urdf/asm_car_asm.urdf.xacro (robot description, xacro)
@@ -4,4 +4,17 @@
      For more information, please see http://wiki.ros.org/sw_urdf_exporter -->
 <robot xmlns:xacro="http://www.ros.org/wiki/xacro" name="asm_car_asm">
+	  <xacro:arg name="transmission_hw_interface" default="hardware_interface/PositionJointInterface"/>
+  <!-- ur5 -->
+  <xacro:include filename="$(find ur_description)/urdf/ur5.urdf.xacro" />
+  <!-- arm -->
+  <xacro:ur5_robot prefix="ur5_" joint_limited="true"
+    shoulder_pan_lower_limit="${-pi}" shoulder_pan_upper_limit="${pi}"
+    shoulder_lift_lower_limit="${-pi}" shoulder_lift_upper_limit="${pi}"
+    elbow_joint_lower_limit="${-pi}" elbow_joint_upper_limit="${pi}"
+    wrist_1_lower_limit="${-pi}" wrist_1_upper_limit="${pi}"
+    wrist_2_lower_limit="${-pi}" wrist_2_upper_limit="${pi}"
+    wrist_3_lower_limit="${-pi}" wrist_3_upper_limit="${pi}"
+    transmission_hw_interface="$(arg transmission_hw_interface)"
+  />
   <include filename="$(find asm_car_asm)/urdf/asm_car_asm.urdf"/>
 <gazebo>

Commit message: aa

File: asm_car_asm/urdf/asm_car_asm.urdf (robot description, URDF)
Before this commit: robot asm_car_asm, 19 links, 19 joints
Links:
- added link camera_link, mass 1e-5; collision box size=0.05 0.20 0.05; visual box size=0.05 0.20 0.05
- added link imu_link, mass 1e-5; collision box size=0.05 0.05 0.05; visual box size=0.05 0.05 0.05
Joints:
- added joint camera_joint: type fixed, parent base_link, child camera_link, origin xyz=0.3 0 0.984 rpy=0 0.2349 0, axis 0 1 0
- added joint imu_joint: type fixed, parent base_link, child imu_link, origin xyz=0.3 0 0.984 rpy=0 0.2349 0, axis 0 1 0

File: asm_car_asm/urdf/asm_car_asm.urdf.xacro (robot description, xacro)
@@ -329,5 +329,90 @@
       </sensor>
   </gazebo>
-<gazebo>
+  <!-- stereo camera -->
+    <gazebo reference="camera_link">
+      <sensor type="multicamera" name="stereocamera">
+        <always_on>true</always_on>
+        <update_rate>20</update_rate>
+        <visualize>false</visualize>
+        <camera name="left">
+          <pose>0 0.10 0 0 0 0</pose>
+          <horizontal_fov>1.5</horizontal_fov>
+          <image>
+            <width>848</width>
+            <height>480</height>
+          </image>
+          <clip>
+            <near>0.01</near>
+            <far>100</far>
+          </clip>
+        </camera>
+        <camera name="right">
+          <pose>0 -0.10 0 0 0 0</pose>
+          <horizontal_fov>1.5</horizontal_fov>
+          <image>
+            <width>848</width>
+            <height>480</height>
+          </image>
+          <clip>
+            <near>0.01</near>
+            <far>100</far>
+          </clip>
+        </camera>
+        <plugin name="stereo_camera_controller" filename="libgazebo_ros_multicamera.so">
+          <cameraName>stereocamera</cameraName>
+          <alwaysOn>true</alwaysOn>
+          <updateRate>20</updateRate>
+          <cameraName>stereocamera</cameraName>
+          <imageTopicName>image_raw</imageTopicName>
+          <cameraInfoTopicName>camera_info</cameraInfoTopicName>
+          <frameName>camera_link_optical</frameName>
+          <baseline>0.20</baseline>
+          <distortion_k1>0.0</distortion_k1>
+          <distortion_k2>0.0</distortion_k2>
+          <distortion_k3>0.0</distortion_k3>
+          <distortion_t1>0.0</distortion_t1>
+          <distortion_t2>0.0</distortion_t2>
+        </plugin>
+      </sensor>
+    </gazebo>
+  <!-- imu -->
+    <!--gazebo reference="imu_link">
+        <gravity>true</gravity>
+        <sensor name="imu" type="imu">
+            <always_on>true</always_on>
+            <update_rate>100</update_rate>
+            <topic>/imu</topic>
+            <plugin name="imu_plugin" filename="libgazebo_ros_imu_sensor.so" >
+                <topicName>/imu</topicName>
+                <bodyName>imu_link</bodyName>
+                <updateRateHZ>100</updateRateHZ>
+                <gaussianNoise>0.01</gaussianNoise>
+                <xyzOffset>0 0 0</xyzOffset>
+                <rpyOffset>0 0 0</rpyOffset>
+                <frameName>imu_link</frameName>
+            </plugin>
+            <pose>0 0 0 0 0 0</pose>
+        </sensor>
+    </gazebo-->
+  <gazebo reference="imu_link">
+    <gravity>true</gravity>
+    <sensor name="imu_sensor" type="imu">
+      <always_on>true</always_on>
+      <update_rate>100</update_rate>
+      <visualize>true</visualize>
+      <topic>__default_topic__</topic>
+      <plugin filename="libgazebo_ros_imu_sensor.so" name="imu_plugin">
+        <topicName>imu</topicName>
+        <bodyName>imu_link</bodyName>
+        <updateRateHZ>100.0</updateRateHZ>
+        <gaussianNoise>0.0</gaussianNoise>
+        <xyzOffset>0 0 0</xyzOffset>
+        <rpyOffset>0 0 0</rpyOffset>
+        <frameName>imu_link</frameName>
+      </plugin>
+      <pose>0 0 0 0 0 0</pose>
+    </sensor>
+  </gazebo>
+  <gazebo>
 	  <plugin name="p3d_base_controller" filename="libgazebo_ros_p3d.so">
 	    <alwaysOn>true</alwaysOn>

File: iqr_4b_robot-master/iqr_4b_description/urdf/iqr_4b_robot.urdf.xacro (robot description, xacro)
@@ -8,5 +8,5 @@
   <xacro:include filename="$(find ${package_name})/urdf/vlp16.xacro"/>
   <xacro:include filename="$(find ${package_name})/urdf/kinect_v2.xacro"/>
-  <xacro:include filename="$(find kinova_description)/urdf/j2n6s300.xacro"/>
+  <!--xacro:include filename="$(find kinova_description)/urdf/j2n6s300.xacro"/-->
   <xacro:include filename="$(find ${package_name})/urdf/jackal_support.xacro"/>
   <xacro:include filename="$(find pan_tilt_description)/urdf/pan_tilt.urdf.xacro" />

File: iqr_4b_robot-master/iqr_4b_description/urdf/kinect_v2.xacro (robot description, xacro)
@@ -26,4 +26,5 @@
     </joint>
     <gazebo reference="${prefix}_link">
+    <plugin name="model_push" filename="libmodel_push.so"/>
     <material>Gazebo/FlatBlack</material>
     <sensor type="depth" name="camera">

Commit message: kinetic 502

File: asm_car_asm/urdf/asm_car_asm.urdf (robot description, URDF)
Before this commit: robot asm_car_asm, 21 links, 21 joints
Links:
- removed link camera_link
Joints:
- removed joint camera_joint
- removed joint ur5_joint
- joint kinect_joint: origin xyz=0 0 0.603 rpy=0 0.7 -1.5708 -> xyz=0 0 0.603 rpy=0 0.2349 -1.5708

File: asm_car_asm/urdf/asm_car_asm.urdf.xacro (robot description, xacro)
@@ -5,7 +5,7 @@
 <robot xmlns:xacro="http://www.ros.org/wiki/xacro" name="asm_car_asm">
 	  <xacro:arg name="transmission_hw_interface" default="hardware_interface/PositionJointInterface"/>
-  <!-- ur5 -->
-  <xacro:include filename="$(find ur_description)/urdf/ur5.urdf.xacro" />
-  <!-- arm -->
+  <!-- ur5 >
+  <xacro:include filename="$(find ur_description)/urdf/ur5.urdf.xacro" /-->
+  <!-- arm >
   <xacro:ur5_robot prefix="ur5_" joint_limited="true"
     shoulder_pan_lower_limit="${-pi}" shoulder_pan_upper_limit="${pi}"
@@ -16,10 +16,11 @@
     wrist_3_lower_limit="${-pi}" wrist_3_upper_limit="${pi}"
     transmission_hw_interface="$(arg transmission_hw_interface)"
-  />
+  /-->
   <include filename="$(find asm_car_asm)/urdf/asm_car_asm.urdf"/>
 <gazebo>
   <plugin name="gazebo_ros_control" filename="libgazebo_ros_control.so">
-    <robotNamespace>/</robotNamespace>
-    <robotSimType>gazebo_ros_control/DefaultRobotHWSim</robotSimType>
+    <!--robotNamespace>/</robotNamespace>
+    <robotSimType>gazebo_ros_control/DefaultRobotHWSim</robotSimType-->
+    <legacyModeNS>true</legacyModeNS>
   </plugin>
 </gazebo>
@@ -330,5 +331,5 @@
   </gazebo>
   <!-- stereo camera -->
-    <gazebo reference="camera_link">
+    <gazebo reference="kinect_link">
       <sensor type="multicamera" name="stereocamera">
         <always_on>true</always_on>
